Commit message: Improved structure and params

File: src/navigation_pkg/urdf/patrol_robot.urdf.xacro (robot description, xacro)
@@ -1,284 +1,168 @@
 <?xml version="1.0"?>
-<robot name="patrol_robot" xmlns:xacro="http://www.ros.org/wiki/xacro">
-  <!-- =========================================================== -->
-  <!--                     PROPERTIES / VARIABLES                   -->
-  <!-- =========================================================== -->
-  <!-- Base link dimensions -->
-  <xacro:property name="base_length"     value="0.7"/>
+<robot xmlns:xacro="http://www.ros.org/wiki/xacro" name="amr_robot">
+  <xacro:property name="base_mass"       value="15.0"/>
+  <xacro:property name="base_length"     value="0.5"/>
   <xacro:property name="base_width"      value="0.4"/>
-  <xacro:property name="base_height"     value="0.2"/>
-  <xacro:property name="base_z_offset"   value="0.1"/>
-  <xacro:property name="base_joint_z"    value="0.05"/>
-  <!-- Drive wheels -->
+  <xacro:property name="base_height"     value="0.1"/>
+  <xacro:property name="wheel_mass"      value="0.8"/>
   <xacro:property name="wheel_radius"    value="0.1"/>
-  <xacro:property name="wheel_length"    value="0.05"/>
-  <xacro:property name="wheel_mass"      value="0.3"/>
-  <xacro:property name="wheel_x_offset"  value="-0.175"/>
-  <xacro:property name="wheel_y_offset"  value="0.225"/>
-  <!-- FIX #1: wheel_separation now matches actual wheel placement (2 * 0.225 = 0.45 m) -->
-  <!-- Previously 0.38 m — mismatched the physical joint positions, causing odometry drift -->
-  <xacro:property name="wheel_separation" value="0.45"/>
-  <xacro:property name="wheel_diameter"  value="${2 * wheel_radius}"/>
-  <!-- Caster wheel -->
-  <xacro:property name="caster_radius"   value="0.05"/>
-  <xacro:property name="caster_mass"     value="0.1"/>
-  <xacro:property name="caster_x_offset" value="0.2"/>
-  <xacro:property name="caster_z_offset" value="-0.05"/>
-  <!-- Camera -->
-  <xacro:property name="camera_size_x"   value="0.05"/>
-  <xacro:property name="camera_size_y"   value="0.10"/>
-  <xacro:property name="camera_size_z"   value="0.05"/>
-  <xacro:property name="camera_mass"     value="0.05"/>
-  <xacro:property name="camera_x"        value="0.30"/>
-  <xacro:property name="camera_y"        value="0.0"/>
-  <xacro:property name="camera_z"        value="0.20"/>
-  <!-- Camera sensor parameters -->
-  <xacro:property name="camera_hz"       value="30"/>
-  <xacro:property name="image_width"     value="640"/>
-  <xacro:property name="image_height"    value="480"/>
-  <xacro:property name="hfov"            value="1.3962634"/>  <!-- 80 degrees -->
-  <xacro:property name="clip_near"       value="0.1"/>
-  <xacro:property name="clip_far"        value="10.0"/>
-  <!-- Lidar -->
-  <xacro:property name="lidar_radius"    value="0.1"/>
-  <xacro:property name="lidar_coll_radius" value="0.05"/>
-  <xacro:property name="lidar_length"    value="0.05"/>
-  <xacro:property name="lidar_mass"      value="0.114"/>
-  <xacro:property name="lidar_z_offset"  value="0.225"/>
-  <!-- Laser scan parameters -->
-  <xacro:property name="laser_samples"   value="720"/>
-  <xacro:property name="laser_min_angle" value="-3.14"/>
-  <xacro:property name="laser_max_angle" value="3.14"/>
-  <xacro:property name="laser_min_range" value="0.1"/>
-  <xacro:property name="laser_max_range" value="12"/>
-  <xacro:property name="laser_range_res" value="0.01"/>
-  <xacro:property name="laser_update_rate" value="10"/>
-  <!-- Joint dynamics -->
-  <xacro:property name="wheel_damping"   value="0.2"/>
-  <xacro:property name="wheel_friction"  value="1.0"/>
-  <xacro:property name="wheel_effort"    value="100"/>
-  <xacro:property name="wheel_velocity"  value="5.0"/>
-  <xacro:property name="caster_damping"  value="0.2"/>
-  <xacro:property name="caster_friction" value="0.1"/>
-  <!-- Diff-drive plugin limits -->
-  <xacro:property name="max_wheel_torque"       value="200"/>
-  <xacro:property name="max_wheel_acceleration" value="10.0"/>
-  <!-- Update rates -->
-  <xacro:property name="imu_update_rate"          value="100"/>
-  <xacro:property name="joint_state_update_rate"  value="30"/>
-  <!-- =========================================================== -->
-  <!--                        MATERIALS                             -->
-  <!-- =========================================================== -->
-  <material name="black">
-    <color rgba="0 0 0 1.0"/>
-  </material>
-  <material name="grey">
-    <color rgba="0.7 0.7 0.7 1.0"/>
-  </material>
-  <material name="green">
-    <color rgba="0.0 0.6 0 1.0"/>
-  </material>
-  <material name="white">
-    <color rgba="1 1 1 1.0"/>
-  </material>
-  <!-- FIX #2: Added missing "blue" material — camera_link referenced it but it was undefined -->
-  <material name="blue">
-    <color rgba="0.0 0.0 0.8 1.0"/>
-  </material>
-  <!-- =========================================================== -->
-  <!--                          LINKS                               -->
-  <!-- =========================================================== -->
+  <xacro:property name="wheel_width"     value="0.05"/>
+  <xacro:property name="wheel_sep"       value="0.45"/>
+  <xacro:property name="caster_radius"   value="0.04"/>
+  <xacro:macro name="box_inertia" params="m x y z">
+    <inertial>
+      <mass value="${m}"/>
+      <inertia
+        ixx="${m/12.0*(y*y+z*z)}" ixy="0.0" ixz="0.0"
+        iyy="${m/12.0*(x*x+z*z)}" iyz="0.0"
+        izz="${m/12.0*(x*x+y*y)}"/>
+    </inertial>
+  </xacro:macro>
+  <xacro:macro name="cylinder_inertia" params="m r h">
+    <inertial>
+      <mass value="${m}"/>
+      <inertia
+        ixx="${m/12.0*(3*r*r+h*h)}" ixy="0.0" ixz="0.0"
+        iyy="${m/12.0*(3*r*r+h*h)}" iyz="0.0"
+        izz="${m/2.0*r*r}"/>
+    </inertial>
+  </xacro:macro>
+  <xacro:macro name="sphere_inertia" params="m r">
+    <inertial>
+      <mass value="${m}"/>
+      <inertia
+        ixx="${2.0/5.0*m*r*r}" ixy="0.0" ixz="0.0"
+        iyy="${2.0/5.0*m*r*r}" iyz="0.0"
+        izz="${2.0/5.0*m*r*r}"/>
+    </inertial>
+  </xacro:macro>
   <link name="base_footprint"/>
+  <joint name="base_joint" type="fixed">
+    <parent link="base_footprint"/>
+    <child  link="base_link"/>
+    <origin xyz="0 0 ${wheel_radius}" rpy="0 0 0"/>
+  </joint>
   <link name="base_link">
-    <inertial>
-      <origin xyz="0.0 0.0 0.0" rpy="0.0 0.0 0.0"/>
-      <mass value="0.1"/>
-      <inertia ixx="0.001665" ixy="0.0" ixz="0.0"
-               iyy="0.00441225" iyz="0.0"
-               izz="0.00541625"/>
-    </inertial>
     <visual>
       <geometry>
         <box size="${base_length} ${base_width} ${base_height}"/>
       </geometry>
-      <origin xyz="0.0 0.0 ${base_z_offset}" rpy="0.0 0.0 0.0"/>
-      <material name="green"/>
-    </visual>
-    <!-- FIX #3: Added missing collision geometry for base_link -->
-    <!-- Without this, Gazebo has no collision body → physics instability → erratic odometry -->
-    <collision>
-      <geometry>
-        <box size="${base_length} ${base_width} ${base_height}"/>
-      </geometry>
-      <origin xyz="0.0 0.0 ${base_z_offset}" rpy="0.0 0.0 0.0"/>
-    </collision>
-  </link>
-  <!-- Left wheel -->
-  <link name="left_wheel">
-    <inertial>
-      <origin xyz="0.0 0.0 0.0" rpy="0.0 0.0 0.0"/>
-      <mass value="${wheel_mass}"/>
-      <inertia ixx="0.00081252" ixy="0.0" ixz="0.0"
-               iyy="0.00081252" iyz="0.0"
-               izz="0.0015"/>
-    </inertial>
-    <visual>
-      <geometry>
-        <cylinder radius="${wheel_radius}" length="${wheel_length}"/>
-      </geometry>
-      <origin xyz="0.0 0.0 0.0" rpy="1.57 0.0 0.0"/>
-      <material name="black"/>
+      <material name="blue">
+        <color rgba="0.15 0.35 0.75 1.0"/>
+      </material>
     </visual>
     <collision>
       <geometry>
-        <cylinder radius="${wheel_radius}" length="${wheel_length}"/>
-      </geometry>
-      <origin xyz="0.0 0.0 0.0" rpy="1.57 0.0 0.0"/>
+        <box size="${base_length} ${base_width} ${base_height}"/>
+      </geometry>
     </collision>
+    <xacro:box_inertia m="${base_mass}" x="${base_length}" y="${base_width}" z="${base_height}"/>
   </link>
-  <!-- Right wheel -->
-  <link name="right_wheel">
-    <inertial>
-      <origin xyz="0.0 0.0 0.0" rpy="0.0 0.0 0.0"/>
-      <mass value="${wheel_mass}"/>
-      <inertia ixx="0.00081252" ixy="0.0" ixz="0.0"
-               iyy="0.00081252" iyz="0.0"
-               izz="0.0015"/>
-    </inertial>
+  <xacro:macro name="drive_wheel" params="prefix y_sign">
+    <link name="${prefix}_wheel">
+      <visual>
+        <origin xyz="0 0 0" rpy="${pi/2} 0 0"/>
+        <geometry>
+          <cylinder radius="${wheel_radius}" length="${wheel_width}"/>
+        </geometry>
+        <material name="dark_gray">
+          <color rgba="0.15 0.15 0.15 1.0"/>
+        </material>
+      </visual>
+      <collision>
+        <origin xyz="0 0 0" rpy="${pi/2} 0 0"/>
+        <geometry>
+          <sphere radius="${wheel_radius}"/>
+        </geometry>
+      </collision>
+      <xacro:cylinder_inertia m="${wheel_mass}" r="${wheel_radius}" h="${wheel_width}"/>
+    </link>
+    <joint name="${prefix}_wheel_joint" type="continuous">
+      <parent link="base_link"/>
+      <child  link="${prefix}_wheel"/>
+      <origin xyz="${-(base_length/2 - 0.1)} ${y_sign * wheel_sep/2} 0" rpy="0 0 0"/>
+      <axis xyz="0 1 0"/>
+    </joint>
+  </xacro:macro>
+  <xacro:drive_wheel prefix="left"  y_sign="1"/>
+  <xacro:drive_wheel prefix="right" y_sign="-1"/>
+  <xacro:macro name="caster" params="prefix x_pos">
+    <link name="${prefix}_caster">
+      <visual>
+        <geometry>
+          <sphere radius="${caster_radius}"/>
+        </geometry>
+        <material name="dark_gray">
+          <color rgba="0.15 0.15 0.15 1.0"/>
+        </material>
+      </visual>
+      <collision>
+        <geometry>
+          <sphere radius="${caster_radius}"/>
+        </geometry>
+      </collision>
+      <xacro:sphere_inertia m="0.1" r="${caster_radius}"/>
+    </link>
+    <joint name="${prefix}_caster_joint" type="fixed">
+      <parent link="base_link"/>
+      <child  link="${prefix}_caster"/>
+      <origin xyz="${x_pos} 0 ${-(base_height/2 + caster_radius - 0.01)}" rpy="0 0 0"/>
+    </joint>
+  </xacro:macro>
+  <xacro:caster prefix="front" x_pos=" ${base_length/2 - 0.06}"/>
+  <link name="lidar_link">
     <visual>
       <geometry>
-        <cylinder radius="${wheel_radius}" length="${wheel_length}"/>
-      </geometry>
-      <origin xyz="0.0 0.0 0.0" rpy="1.57 0.0 0.0"/>
-      <material name="black"/>
+        <cylinder radius="0.04" length="0.06"/>
+      </geometry>
+      <material name="black">
+        <color rgba="0.05 0.05 0.05 1.0"/>
+      </material>
     </visual>
     <collision>
       <geometry>
-        <cylinder radius="${wheel_radius}" length="${wheel_length}"/>
-      </geometry>
-      <origin xyz="0.0 0.0 0.0" rpy="1.57 0.0 0.0"/>
+        <cylinder radius="0.04" length="0.06"/>
+      </geometry>
     </collision>
+    <inertial>
+      <mass value="0.1"/>
+      <inertia ixx="0.001" ixy="0" ixz="0" iyy="0.001" iyz="0" izz="0.001"/>
+    </inertial>
   </link>
-  <!-- Caster wheel -->
-  <link name="caster_wheel">
-    <inertial>
-      <origin xyz="0.0 0.0 0.0" rpy="0.0 0.0 0.0"/>
-      <mass value="${caster_mass}"/>
-      <inertia ixx="0.00016666" ixy="0.0" ixz="0.0"
-               iyy="0.00016666" iyz="0.0"
-               izz="0.00016666"/>
-    </inertial>
+  <joint name="lidar_joint" type="fixed">
+    <parent link="base_link"/>
+    <child  link="lidar_link"/>
+    <origin xyz="0 0 ${base_height/2 + 0.03}" rpy="0 0 0"/>
+  </joint>
+  <link name="camera_link">
     <visual>
       <geometry>
-        <sphere radius="${caster_radius}"/>
-      </geometry>
-      <origin xyz="0.0 0.0 0.0" rpy="0.0 0.0 0.0"/>
-      <material name="black"/>
+        <box size="0.04 0.08 0.04"/>
+      </geometry>
+      <material name="dark_gray">
+        <color rgba="0.25 0.25 0.25 1.0"/>
+      </material>
     </visual>
     <collision>
       <geometry>
-        <sphere radius="${caster_radius}"/>
-      </geometry>
-      <origin xyz="0.0 0.0 0.0" rpy="0.0 0.0 0.0"/>
+        <box size="0.04 0.08 0.04"/>
+      </geometry>
     </collision>
+    <inertial>
+      <mass value="0.05"/>
+      <inertia ixx="0.0001" ixy="0" ixz="0" iyy="0.0001" iyz="0" izz="0.0001"/>
+    </inertial>
   </link>
-  <link name="camera_link">
-    <visual>
-      <geometry>
-        <box size="${camera_size_x} ${camera_size_y} ${camera_size_z}"/>
-      </geometry>
-      <origin xyz="0 0 0" rpy="0 0 0"/>
-      <!-- FIX #2 (applied): now uses defined "blue" material -->
-      <material name="blue"/>
-    </visual>
-    <collision>
-      <geometry>
-        <box size="${camera_size_x} ${camera_size_y} ${camera_size_z}"/>
-      </geometry>
-      <origin xyz="0 0 0" rpy="0 0 0"/>
-    </collision>
-    <inertial>
-      <mass value="${camera_mass}"/>
-      <origin xyz="0 0 0"/>
-      <inertia ixx="2.08e-5" ixy="0.0" ixz="0.0"
-               iyy="2.08e-5" iyz="0.0"
-               izz="2.08e-5"/>
-    </inertial>
-  </link>
-  <link name="camera_link_optical"/>
-  <!-- Lidar -->
-  <link name="lidar_link">
-    <visual>
-      <geometry>
-        <cylinder radius="${lidar_radius}" length="${lidar_length}"/>
-      </geometry>
-      <origin xyz="0.0 0.0 0.0" rpy="0.0 0.0 0.0"/>
-      <material name="white"/>
-    </visual>
-    <collision>
-      <geometry>
-        <cylinder radius="${lidar_coll_radius}" length="${lidar_length}"/>
-      </geometry>
-      <origin xyz="0.0 0.0 0.0" rpy="0.0 0.0 0.0"/>
-    </collision>
-    <inertial>
-      <mass value="${lidar_mass}"/>
-      <origin xyz="0 0 0"/>
-      <inertia ixx="0.001" ixy="0.0" ixz="0.0"
-               iyy="0.001" iyz="0.0"
-               izz="0.001"/>
-    </inertial>
-  </link>
-  <!-- =========================================================== -->
-  <!--                          JOINTS                              -->
-  <!-- =========================================================== -->
-  <joint name="base_joint" type="fixed">
-    <parent link="base_footprint"/>
-    <child link="base_link"/>
-    <origin xyz="0.0 0.0 ${base_joint_z}" rpy="0.0 0.0 0.0"/>
-  </joint>
-  <joint name="base_lidar_joint" type="fixed">
-    <parent link="base_link"/>
-    <child link="lidar_link"/>
-    <origin xyz="0.0 0.0 ${lidar_z_offset}" rpy="0.0 0.0 0.0"/>
-  </joint>
-  <joint name="left_wheel_joint" type="continuous">
-    <parent link="base_link"/>
-    <child link="left_wheel"/>
-    <origin xyz="${wheel_x_offset} ${wheel_y_offset} 0.0" rpy="0 0.0 0.0"/>
-    <axis xyz="0.0 1.0 0.0"/>
-    <dynamics damping="${wheel_damping}" friction="${wheel_friction}"/>
-    <limit effort="${wheel_effort}" velocity="${wheel_velocity}"/>
-  </joint>
-  <joint name="right_wheel_joint" type="continuous">
-    <parent link="base_link"/>
-    <child link="right_wheel"/>
-    <origin xyz="${wheel_x_offset} -${wheel_y_offset} 0.0" rpy="0 0.0 0.0"/>
-    <axis xyz="0.0 1.0 0.0"/>
-    <dynamics damping="${wheel_damping}" friction="${wheel_friction}"/>
-    <limit effort="${wheel_effort}" velocity="${wheel_velocity}"/>
-  </joint>
-  <joint name="caster_wheel_joint" type="fixed">
-    <parent link="base_link"/>
-    <child link="caster_wheel"/>
-    <dynamics damping="${caster_damping}" friction="${caster_friction}"/>
-    <origin xyz="${caster_x_offset} 0.0 ${caster_z_offset}" rpy="0.0 0.0 0.0"/>
-  </joint>
   <joint name="camera_joint" type="fixed">
     <parent link="base_link"/>
     <child  link="camera_link"/>
-    <origin xyz="${camera_x} ${camera_y} ${camera_z}" rpy="0.0 0.0 0.0"/>
-  </joint>
-  <!-- Camera optical frame joint — pure rotation for ROS convention -->
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
Commit message: Improved structure and params

File: src/navigation_pkg/urdf/patrol_robot.urdf.xacro (robot description, xacro)
@@ -9,5 +9,20 @@
   <xacro:property name="wheel_width"     value="0.05"/>
   <xacro:property name="wheel_sep"       value="0.45"/>
+  <xacro:property name="wheel_x_offset"  value="0.1"/>
+  <xacro:property name="wheel_damping"   value="0.1"/>
+  <xacro:property name="wheel_friction"  value="0.0"/>
+  <xacro:property name="wheel_effort"    value="10.0"/>
+  <xacro:property name="wheel_velocity"  value="5.0"/>
   <xacro:property name="caster_radius"   value="0.04"/>
+  <xacro:property name="caster_mass"     value="0.1"/>
+  <xacro:property name="caster_z"        value="${-(wheel_radius - caster_radius)}"/>
+  <xacro:property name="caster_x_reach"  value="${base_length/2 - 0.06}"/>
+  <xacro:property name="lidar_radius"    value="0.04"/>
+  <xacro:property name="lidar_length"    value="0.06"/>
+  <xacro:property name="lidar_mass"      value="0.1"/>
+  <xacro:property name="camera_size_x"   value="0.04"/>
+  <xacro:property name="camera_size_y"   value="0.08"/>
+  <xacro:property name="camera_size_z"   value="0.04"/>
+  <xacro:property name="camera_mass"     value="0.05"/>
   <xacro:macro name="box_inertia" params="m x y z">
     <inertial>
@@ -73,5 +88,5 @@
         <origin xyz="0 0 0" rpy="${pi/2} 0 0"/>
         <geometry>
-          <sphere radius="${wheel_radius}"/>
+          <cylinder radius="${wheel_radius}" length="${wheel_width}"/>
         </geometry>
       </collision>
@@ -81,6 +96,8 @@
       <parent link="base_link"/>
       <child  link="${prefix}_wheel"/>
-      <origin xyz="${-(base_length/2 - 0.1)} ${y_sign * wheel_sep/2} 0" rpy="0 0 0"/>
+      <origin xyz="${-(base_length/2 - wheel_x_offset)} ${y_sign * wheel_sep/2} 0" rpy="0 0 0"/>
       <axis xyz="0 1 0"/>
+      <dynamics damping="${wheel_damping}" friction="${wheel_friction}"/>
+      <limit effort="${wheel_effort}" velocity="${wheel_velocity}"/>
     </joint>
   </xacro:macro>
@@ -102,17 +119,18 @@
         </geometry>
       </collision>
-      <xacro:sphere_inertia m="0.1" r="${caster_radius}"/>
+      <xacro:sphere_inertia m="${caster_mass}" r="${caster_radius}"/>
     </link>
     <joint name="${prefix}_caster_joint" type="fixed">
       <parent link="base_link"/>
       <child  link="${prefix}_caster"/>
-      <origin xyz="${x_pos} 0 ${-(base_height/2 + caster_radius - 0.01)}" rpy="0 0 0"/>
+      <origin xyz="${x_pos} 0 ${caster_z}" rpy="0 0 0"/>
     </joint>
   </xacro:macro>
-  <xacro:caster prefix="front" x_pos=" ${base_length/2 - 0.06}"/>
+  <xacro:caster prefix="front" x_pos="${caster_x_reach}"/>
+  <xacro:caster prefix="rear"  x_pos="${-caster_x_reach}"/>
   <link name="lidar_link">
     <visual>
       <geometry>
-        <cylinder radius="0.04" length="0.06"/>
+        <cylinder radius="${lidar_radius}" length="${lidar_length}"/>
       </geometry>
       <material name="black">
@@ -122,21 +140,18 @@
     <collision>
       <geometry>
-        <cylinder radius="0.04" length="0.06"/>
+        <cylinder radius="${lidar_radius}" length="${lidar_length}"/>
       </geometry>
     </collision>
-    <inertial>
-      <mass value="0.1"/>
-      <inertia ixx="0.001" ixy="0" ixz="0" iyy="0.001" iyz="0" izz="0.001"/>
-    </inertial>
+    <xacro:cylinder_inertia m="${lidar_mass}" r="${lidar_radius}" h="${lidar_length}"/>
   </link>
   <joint name="lidar_joint" type="fixed">
     <parent link="base_link"/>
     <child  link="lidar_link"/>
-    <origin xyz="0 0 ${base_height/2 + 0.03}" rpy="0 0 0"/>
+    <origin xyz="0 0 ${base_height/2 + lidar_length/2}" rpy="0 0 0"/>
   </joint>
   <link name="camera_link">
     <visual>
       <geometry>
-        <box size="0.04 0.08 0.04"/>
+        <box size="${camera_size_x} ${camera_size_y} ${camera_size_z}"/>
       </geometry>
       <material name="dark_gray">
@@ -146,11 +161,11 @@
     <collision>
       <geometry>
-        <box size="0.04 0.08 0.04"/>
+        <box size="${camera_size_x} ${camera_size_y} ${camera_size_z}"/>
       </geometry>
     </collision>
-    <inertial>
-      <mass value="0.05"/>
-      <inertia ixx="0.0001" ixy="0" ixz="0" iyy="0.0001" iyz="0" izz="0.0001"/>
-    </inertial>
+    <xacro:box_inertia m="${camera_mass}"
+                       x="${camera_size_x}"
+                       y="${camera_size_y}"
+                       z="${camera_size_z}"/>
   </link>
   <joint name="camera_joint" type="fixed">
@@ -224,5 +239,5 @@
       <gz_frame_id>camera_optical_frame</gz_frame_id>
       <camera>
-        <horizontal_fov>1.047</horizontal_fov>  <!-- 60 degrees -->
+        <horizontal_fov>1.047</horizontal_fov> <!-- 60 degrees -->
         <image>
           <width>640</width>
@@ -239,4 +254,13 @@
     </sensor>
   </gazebo>
+  <gazebo reference="base_link">
+    <material>Gazebo/Blue</material>
+  </gazebo>
+  <gazebo reference="lidar_link">
+    <material>Gazebo/Black</material>
+  </gazebo>
+  <gazebo reference="camera_link">
+    <material>Gazebo/DarkGrey</material>
+  </gazebo>
   <gazebo reference="left_wheel">
     <mu1>1.0</mu1>

Commit message: Corrected state machine.

File: src/navigation_pkg/urdf/patrol_robot.urdf.xacro (robot description, xacro)
@@ -63,5 +63,5 @@
         <box size="${base_length} ${base_width} ${base_height}"/>
       </geometry>
-      <material name="blue">
+      <material name="red">
         <color rgba="0.15 0.35 0.75 1.0"/>
       </material>
@@ -255,5 +255,5 @@
   </gazebo>
   <gazebo reference="base_link">
-    <material>Gazebo/Blue</material>
+    <material>Gazebo/Red</material>
   </gazebo>
   <gazebo reference="lidar_link">
